File: pcb/TempMonitorPCB/tempmon/tempmon.kicad_pcb (KiCad board)
At the start: 2 copper layers, 5 parts, among them J1 USB_A, U1 ENS210, U2 WeMos_D1_mini

Commit message: Routing Complete :)
I hope it is at least, I barely know how to make PCBs
Routing:
- net GND: track 28.8 -> 69.6 mm, vias 0 -> 1
- net /pull-up-sda: track 17.8 -> 19.4 mm, vias 1 -> 2
- net (no net): vias 1 -> 0
Other:
- board outline added: 61 x 62 mm
Changed lines of the file:
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@@
 		(tags "QFN 0.95")
 		(property "Reference" "U1"
-			(at 0 -2 360)
+			(at 0 -2 0)
 			(layer "F.SilkS")
 			(effects
@@
 		)
 		(property "Value" "ENS210"
-			(at 0 2 360)
+			(at 0 2 0)
 			(layer "F.Fab")
 			(effects
@@
 		)
 		(fp_text user "${REFERENCE}"
-			(at 0 0 360)
+			(at 0 0 0)
 			(layer "F.Fab")
 			(effects
@@
 		(tags "USB SMD Type-A Receptacle Right Angle")
 		(property "Reference" "J1"
-			(at 0 -10 360)
+			(at 0 -10 0)
 			(layer "F.SilkS")
 			(effects
@@
 		)
 		(property "Value" "USB_A"
-			(at 0 8.5 360)
+			(at 0 8.5 0)
 			(layer "F.Fab")
 			(effects
@@
 		)
 		(fp_text user "PCB Edge"
-			(at 0 4.97 360)
+			(at 0 4.97 0)
 			(layer "Dwgs.User")
 			(effects
@@
 		)
 	)
+	(gr_rect
+		(start 107 46)
+		(end 168 108)
+		(stroke
+			(width 0.05)
+			(type default)
+		)
+		(fill none)
+		(layer "Edge.Cuts")
+	)
 	(segment
 		(start 142.23 87.23)
@@
 		(net 0)
 	)
-	(via
-		(at 147.5 85.5)
-		(size 0.6)
-		(drill 0.3)
-		(layers "F.Cu" "B.Cu")
-		(net 0)
+	(segment
+		(start 146.475 85.475)
+		(end 146.5 85.5)
+		(width 0.2)
+		(layer "F.Cu")
+		(net 1)
 	)
 	(segment
@@
 		(net 1)
 	)
+	(segment
+		(start 144.95 85.475)
+		(end 146.475 85.475)
+		(width 0.2)
+		(layer "F.Cu")
+		(net 1)
+	)
 	(via
 		(at 150 82)
@@
 		(net 1)
 	)
+	(via
+		(at 146.5 85.5)
+		(size 0.6)
+		(drill 0.3)
+		(layers "F.Cu" "B.Cu")
+		(net 1)
+	)
+	(segment
+		(start 150 82)
+		(end 146.5 85.5)
+		(width 0.2)
+		(layer "B.Cu")
+		(net 1)
+	)
+	(segment
+		(start 146 86)
+		(end 145.77 86.23)
+		(width 0.2)
+		(layer "B.Cu")
+		(net 1)
+	)
 	(segment
 		(start 145.77 86.23)
@@
 	)
 	(segment
-		(start 150 82)
-		(end 145.77 86.23)
+		(start 146.5 85.5)
+		(end 146 86)
 		(width 0.2)
 		(layer "B.Cu")
@@
 	)
 	(segment
+		(start 123.9 62.4)
+		(end 123.9 58.7)
+		(width 0.2)
+		(layer "F.Cu")
+		(net 2)
+	)
+	(segment
 		(start 150.85 93.85)
 		(end 137.58 93.85)
@@
 	)
 	(segment
+		(start 124 62.5)
+		(end 123.9 62.4)
+		(width 0.2)
+		(layer "F.Cu")
+		(net 2)
+	)
+	(segment
 		(start 151 93.7)
 		(end 150.85 93.85)
@@
 		(net 2)
 	)
+	(via
+		(at 124 62.5)
+		(size 0.6)
+		(drill 0.3)
+		(layers "F.Cu" "B.Cu")
+		(net 2)
+	)
+	(segment
+		(start 137.58 93.85)
+		(end 124 80.27)
+		(width 0.2)
+		(layer "B.Cu")
+		(net 2)
+	)
+	(segment
+		(start 124 80.27)
+		(end 124 62.5)
+		(width 0.2)
+		(layer "B.Cu")
+		(net 2)
+	)

Commit message: final PCB commit
not on hakkuun
Routing:
- net GND: track 69.6 -> 53.5 mm
- net (no net): track 5.74 -> 0.00 mm
Changed lines of the file:
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@@
-	)
-	(segment
-		(start 142.23 87.23)
-		(end 143 88)
-		(width 0)
-		(layer "F.Cu")
-		(net 0)
-	)
-	(segment
-		(start 142.23 87.23)
-		(end 137.58 87.23)
-		(width 0)
-		(layer "F.Cu")
-		(net 0)
 	)
 	(segment
@@
 	)
 	(segment
-		(start 149.95 84.05)
-		(end 146.9 84.05)
-		(width 0.2)
-		(layer "F.Cu")
-		(net 2)
-	)
-	(segment
 		(start 123.9 62.4)
 		(end 123.9 58.7)
@@
 	)
 	(segment
-		(start 150.85 93.85)
-		(end 137.58 93.85)
+		(start 137.58 93.85)
+		(end 144 87.43)
 		(width 0.2)
 		(layer "F.Cu")
@@
 	)
 	(segment
-		(start 146.9 84.05)
-		(end 146.425 84.525)
+		(start 144.95 84.525)
+		(end 144.475 84.525)
 		(width 0.2)
 		(layer "F.Cu")
@@
 	)
 	(segment
-		(start 151 93.7)
-		(end 150.85 93.85)
+		(start 144 87.43)
+		(end 144 85)
 		(width 0.2)
 		(layer "F.Cu")
@@
 	)
 	(segment
-		(start 151 85.1)
-		(end 149.95 84.05)
+		(start 144.475 84.525)
+		(end 144 85)
 		(width 0.2)
 		(layer "F.Cu")
-		(net 2)
-	)
-	(segment
-		(start 151 93.7)
-		(end 151 85.1)
-		(width 0.2)
-		(layer "F.Cu")
-		(net 2)
-	)
-	(segment
-		(start 146.425 84.525)
-		(end 144.95 84.525)
-		(width 0.2)
-		(layer "F.Cu")
